File: Pi Button.kicad_sch (KiCad schematic)
At the start: 5 parts, among them J1 Conn_02x20_Odd_Even, SW1 SW_Push, SW2 SW_Push

Commit message: part placement
Parts:
- R1, R2: footprint Resistor_SMD:R_0805_2012Metric -> Resistor_THT:R_Axial_DIN0204_L3.6mm_D1.6mm_P2.54mm_Vertical
Other:
- company: (none) -> Aero Scan
- title: (none) -> Button PCB
Changed lines of the file:
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@@
 	(generator_version "9.0")
 	(paper "A4")
+	(title_block
+		(title "Button PCB")
+		(date "2025-04-22")
+		(rev "1")
+		(company "Aero Scan")
+	)
 	(junction
 		(at 125.73 72.39)
@@
 			)
 		)
-		(property "Footprint" "Resistor_SMD:R_0805_2012Metric"
+		(property "Footprint" "Resistor_THT:R_Axial_DIN0204_L3.6mm_D1.6mm_P2.54mm_Vertical"
 			(at 171.45 69.088 90)
 			(effects
@@
 			)
 		)
-		(property "Footprint" "Resistor_SMD:R_0805_2012Metric"
+		(property "Footprint" "Resistor_THT:R_Axial_DIN0204_L3.6mm_D1.6mm_P2.54mm_Vertical"
 			(at 171.45 76.708 90)
 			(effects
